File: RIAA_Template.kicad_pcb (KiCad board)
At the start: 2 copper layers, 65 x 39 mm, 34 parts, among them U1 NE5532

Commit message: Updating template with correct dimensions & annotations
Parts:
- removed C11, C15, C21, C25: 10u, Capacitors_ThroughHole:C_Radial_D5_L11_P2.5
- removed C12, C22: 100u, Capacitors_ThroughHole:C_Radial_D5_L11_P2.5
- removed C13, C23: 8n2, Capacitors_ThroughHole:C_Rect_L7_W2.5_P5
- removed C14, C24: 22n, Capacitors_ThroughHole:C_Rect_L7_W2.5_P5
- removed H13, H23: Header_01x03, Pin_Headers:Pin_Header_Straight_1x03
- removed R11, R21: 100, Resistors_ThroughHole:Resistor_Horizontal_RM10mm
- removed R12, R19, R22, R29: 47K, Resistors_ThroughHole:Resistor_Horizontal_RM10mm
- removed R13, R23: 470, Resistors_ThroughHole:Resistor_Horizontal_RM10mm
- removed R14, R24: 10K, Resistors_ThroughHole:Resistor_Horizontal_RM10mm
- removed R15, R25: 150, Resistors_ThroughHole:Resistor_Horizontal_RM10mm
- removed R17, R27: 100K, Resistors_ThroughHole:Resistor_Horizontal_RM10mm
- removed R18, R28: 1K, Resistors_ThroughHole:Resistor_Horizontal_RM10mm
- removed U1: NE5532, Housings_DIP:DIP-8_W7.62mm_LongPads
Routing:
- net Net-(C15-Pad1): track 59.3 -> 0.00 mm
- net Net-(C25-Pad1): track 57.4 -> 0.00 mm
- net GND: track 38.3 -> 0.00 mm
- net Net-(H23-Pad3): track 32.3 -> 0.00 mm
- net Net-(H13-Pad3): track 32.2 -> 0.00 mm
- net /V-: track 29.5 -> 0.00 mm
- net Net-(C14-Pad1): track 22.0 -> 0.00 mm
- net Net-(C24-Pad1): track 21.1 -> 0.00 mm
- net Net-(R24-Pad2): track 20.1 -> 0.00 mm
- net /V+: track 19.4 -> 0.00 mm
- net Net-(R14-Pad2): track 16.7 -> 0.00 mm
- net Net-(C25-Pad2): track 13.4 -> 0.00 mm
- net Net-(C15-Pad2): track 13.4 -> 0.00 mm
- net Net-(C22-Pad1): track 12.4 -> 0.00 mm
- net Net-(C21-Pad1): track 12.2 -> 0.00 mm
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Other:
- board text added: "GND"
- board text added: "IN_L+"
- board text added: "IN_L-"
- board text added: "IN_R+"
- board text added: "IN_R-"
- board text added: "OUT_L+"
- board text added: "OUT_L-"
- board text added: "OUT_R+"
- board text added: "OUT_R-"
- board text added: "PWR"
- board text added: "V+"
- board text added: "V-"
